File: untitled.brd (EAGLE design)
At the start: 100.3 x 100 mm, 7 parts

Commit message: Add files via upload
Parts:
- removed MPU: (no value), MIA_LIBRARY-2-2-2:1X04_DATA
- added U$2: IMU_ROBOCON_GY521, MIA_LIBRARY-2-2-2:IMU_GY521
- TTL1, TTL2: device MIA_LIBRARY-2-2-2:1X04_DATA -> MIA_LIBRARY-2-2-2:1X04
- moved TTL1 5.84 mm to (9.00, 31.0)
- moved TTL2 4.96 mm to (77.0, 45.0), turned to 270 degrees
- moved U$1 4.00 mm to (10.3, 45.7)
Connections:
- new net GND_1: DATABASE.1, TTL1.1, U$1.2, U$3.GND_2
- new net GND_3: U$3.GND_3
- net 3.3V1: now also U$2.VCC; no longer MPU.1
- net GND: now also U$2.GND; no longer DATABASE.1, MPU.2, TTL1.1, U$1.2, U$3.GND_2, U$3.GND_3
- net PA_10: now also TTL2.3; no longer TTL2.4
- net PA_9: now also TTL2.4; no longer TTL2.3
- net PB_10: now also TTL1.4; no longer TTL1.3
- net PB_11: now also TTL1.3; no longer TTL1.4
- net PB_6: now also U$2.SCL; no longer MPU.3
- net PB_7: now also U$2.SDA; no longer MPU.4
Routing:
- net GND: track 411.8 -> 88.6 mm, vias 4 -> 0
- net PB_7: track 111.5 -> 17.4 mm, vias 2 -> 0
- net GND_1: track 0.00 -> 88.7 mm, vias 0 -> 2
- net 5V: track 308.3 -> 270.9 mm, vias 2 -> 3
- net PB_10: track 53.2 -> 21.0 mm, vias 2 -> 0
- net 3.3V1: track 33.9 -> 15.8 mm, vias 2 -> 0
- net PB_6: track 28.1 -> 40.3 mm
- net PB_11: track 28.9 -> 21.0 mm
- net PB_1: track 23.9 -> 19.9 mm
- net PB_0: track 23.9 -> 19.9 mm
- net PA_10: track 31.1 -> 35.0 mm
- net PA_9: track 31.1 -> 34.4 mm
