File: untitled.sch (EAGLE design)
At the start: 7 parts

Commit message: Add files via upload
Parts:
- removed MPU: (no value), MIA_LIBRARY-2-2-2:PINHD-4_DATA
- added U$2: IMU_ROBOCON_GY521, MIA_LIBRARY-2-2-2:IMU_ROBOCON_GY521
- TTL1, TTL2: device MIA_LIBRARY-2-2-2:I2C_LCD_STANDARD -> MIA_LIBRARY-2-2-2:PINHD-1X4
Connections:
- new net GND_1: DATABASE.1, TTL1.1, U$1.GND, U$3.GND@2
- new net GND_3: U$3.GND@3
- net 3.3V1: now also U$2.VCC; no longer MPU.1
- net GND: now also U$2.GND; no longer DATABASE.1, MPU.2, TTL1.1, U$1.GND, U$3.GND@2, U$3.GND@3
- net PA_10: now also TTL2.3; no longer TTL2.4
- net PA_9: now also TTL2.4; no longer TTL2.3
- net PB_10: now also TTL1.4; no longer TTL1.3
- net PB_11: now also TTL1.3; no longer TTL1.4
- net PB_6: now also U$2.SCL; no longer MPU.3
- net PB_7: now also U$2.SDA; no longer MPU.4
